Commit message: Removed T265 support along with the realsense-ros package in lunabot_external. Changed ekf_yaml to use D456 IMU. Cleaned up robot_controller.cpp. Added setup for udev rules for D456 camera. Added realistic arena world for Gazebo. Created keyboard teleop node for controlling robot in Gazebo. Created topic remapping node for ros2_control controller topics. Improved folder structure in lunabot_autonomous.

File: lunabot_description/urdf/common_properties.xacro (robot description, xacro)
@@ -13,5 +13,5 @@
         <color rgba="0.89 0.89 0.89 1.0" />
     </material>
-     <material name="green">
+    <material name="green">
         <color rgba="0.03529412 0.32156863 0.24313725 1.0" />
     </material>

File: lunabot_description/urdf/sim_bot.xacro (robot description, xacro)
@@ -1,6 +1,6 @@
 <?xml version="1.0"?>
-<robot name="sim_bot" xmlns:xacro="http://www.ros.org/wiki/xacro">
+<robot name="sim_bot"
+  xmlns:xacro="http://www.ros.org/wiki/xacro">
   <xacro:include filename="common_properties.xacro" />
-  <!-- Base Link -->
   <link name="base_link">
     <visual>
@@ -11,5 +11,5 @@
       <material name="light_grey" />
     </visual>
-        <collision>
+    <collision>
       <geometry>
         <mesh filename="file:///$(find lunabot_description)/meshes/base_link.stl" />
@@ -17,14 +17,14 @@
       <origin xyz="0 0 0.085" rpy="0 0 0" />
     </collision>
-      <inertial>
-    <mass value="5.0" />
-    <origin xyz="0 0 0.085" />
-    <inertia ixx="0.0833" ixy="0.0" ixz="0.0" iyy="0.1667" iyz="0.0" izz="0.2333" />
-  </inertial>
+    <inertial>
+      <mass value="25.0" />
+      <origin xyz="0 0 0.085" />
+      <inertia ixx="1.3669" ixy="0.0" ixz="0.0" iyy="3.3602" iyz="0.0" izz="4.7271" />
+    </inertial>
   </link>
   <gazebo reference="base_link">
     <material>Gazebo/Grey</material>
   </gazebo>
-    <link name="ebox_link">
+  <link name="ebox_link">
     <visual>
       <geometry>
@@ -34,5 +34,5 @@
       <material name="white" />
     </visual>
-        <collision>
+    <collision>
       <geometry>
         <mesh filename="file:///$(find lunabot_description)/meshes/ebox_link.stl" />
@@ -44,13 +44,13 @@
     <material>Gazebo/White</material>
   </gazebo>
-    <link name="nuc_link">
+  <link name="nuc_link">
     <visual>
       <geometry>
         <mesh filename="file:///$(find lunabot_description)/meshes/nuc_link.stl" />
       </geometry>
-	    <origin xyz="0 0 0" rpy="${pi} 0 ${pi}" />
+      <origin xyz="0 0 0" rpy="${pi} 0 ${pi}" />
       <material name="black" />
     </visual>
-           <collision>
+    <collision>
       <geometry>
         <mesh filename="file:///$(find lunabot_description)/meshes/nuc_link.stl" />
@@ -62,5 +62,5 @@
     <material>Gazebo/Black</material>
   </gazebo>
-    <link name="lidar1_link">
+  <link name="lidar1_link">
     <visual>
       <geometry>
@@ -70,5 +70,5 @@
       <material name="black" />
     </visual>
-      <collision>
+    <collision>
       <geometry>
         <mesh filename="file:///$(find lunabot_description)/meshes/lidar1_link.stl" />
@@ -77,5 +77,28 @@
     </collision>
   </link>
-      <link name="lidar2_link">
+  <link name="blade_link">
+    <visual>
+      <geometry>
+        <mesh filename="file:///$(find lunabot_description)/meshes/blade_link.stl" />
+      </geometry>
+      <origin xyz="0 0 0" rpy="0 0 0" />
+      <material name="light_grey" />
+    </visual>
+    <collision>
+      <geometry>
+        <mesh filename="file:///$(find lunabot_description)/meshes/blade_link.stl" />
+      </geometry>
+      <origin xyz="0 0 0" rpy="0 0 0" />
+    </collision>
+    <inertial>
+      <mass value="5.0" />
+      <origin xyz="0 0 0" />
+      <inertia ixx="0.0833" ixy="0.0" ixz="0.0" iyy="0.1667" iyz="0.0" izz="0.2333" />
+    </inertial>
+  </link>
+  <gazebo reference="blade_link">
+    <material>Gazebo/Grey</material>
+  </gazebo>
+  <link name="lidar2_link">
     <visual>
       <geometry>
@@ -85,5 +108,5 @@
       <material name="black" />
     </visual>
-          <collision>
+    <collision>
       <geometry>
         <mesh filename="file:///$(find lunabot_description)/meshes/lidar2_link.stl" />
@@ -92,21 +115,20 @@
     </collision>
   </link>
-      <link name="d455_link">
+  <link name="d455_link">
     <visual>
       <geometry>
         <mesh filename="file:///$(find lunabot_description)/meshes/camera_link.stl" />
       </geometry>
-      <origin xyz="0 -0.1 0" rpy="0 0 0" />
+      <origin xyz="0 0 0" rpy="0 0 0" />
       <material name="camera_grey" />
     </visual>
-          <collision>
+    <collision>
       <geometry>
         <mesh filename="file:///$(find lunabot_description)/meshes/camera_link.stl" />
       </geometry>
-      <origin xyz="0 -0.1 0" rpy="0 0 0" />
+      <origin xyz="0 0 0" rpy="0 0 0" />
     </collision>
   </link>
   <link name="d455_link_optical"></link>
-  <!-- Wheel Links -->
   <link name="front_right_wheel_link">
     <visual>
@@ -118,9 +140,9 @@
     </visual>
     <inertial>
-      <mass value="0.1" />
+      <mass value="2.27" />
       <origin xyz="0 0 0" />
-      <inertia ixx="0.01" ixy="0.0" ixz="0.0" iyy="0.01" iyz="0.0" izz="0.01" />
-    </inertial>
-          <collision>
+      <inertia ixx="0.0255" ixy="0.0" ixz="0.0"
+        iyy="0.0255" iyz="0.0" izz="0.0510" />> </inertial>
+    <collision>
       <geometry>
         <mesh filename="file:///$(find lunabot_description)/meshes/wheel_link.stl" />
@@ -129,8 +151,20 @@
     </collision>
   </link>
-    <gazebo reference="front_right_wheel_link">
+  <gazebo reference="front_right_wheel_link">
     <material>Gazebo/DarkGrey</material>
-  </gazebo>
-    <link name="front_left_wheel_link">
+    <mu>1.0</mu>
+    <mu2>1.0</mu2>
+    <surface>
+      <contact>
+        <ode>
+          <kp>1000000</kp>
+          <kd>500</kd>
+          <slip1>0.02</slip1>
+          <slip2>0.02</slip2>
+        </ode>
+      </contact>
+    </surface>
+  </gazebo>
+  <link name="front_left_wheel_link">
     <visual>
       <geometry>
@@ -141,9 +175,9 @@
     </visual>
     <inertial>
-      <mass value="0.1" />
+      <mass value="2.27" />
       <origin xyz="0 0 0" />
-      <inertia ixx="0.01" ixy="0.0" ixz="0.0" iyy="0.01" iyz="0.0" izz="0.01" />
+      <inertia ixx="0.0255" ixy="0.0" ixz="0.0" iyy="0.0255" iyz="0.0" izz="0.0510" />
     </inertial>
-      <collision>
+    <collision>
       <geometry>
         <mesh filename="file:///$(find lunabot_description)/meshes/wheel_link.stl" />
@@ -152,8 +186,20 @@
     </collision>
   </link>
-    <gazebo reference="front_left_wheel_link">
+  <gazebo reference="front_left_wheel_link">
     <material>Gazebo/DarkGrey</material>
-  </gazebo>
-    <link name="rear_right_wheel_link">
+    <mu>1.0</mu>
+    <mu2>1.0</mu2>
+    <surface>
+      <contact>
+        <ode>
+          <kp>1000000</kp>
+          <kd>500</kd>
+          <slip1>0.02</slip1>
+          <slip2>0.02</slip2>
+        </ode>
+      </contact>
+    </surface>
+  </gazebo>
+  <link name="rear_right_wheel_link">
     <visual>
       <geometry>
@@ -164,9 +210,9 @@
     </visual>
     <inertial>
-      <mass value="0.1" />
+      <mass value="2.27" />
       <origin xyz="0 0 0" />
-      <inertia ixx="0.01" ixy="0.0" ixz="0.0" iyy="0.01" iyz="0.0" izz="0.01" />
+      <inertia ixx="0.0255" ixy="0.0" ixz="0.0" iyy="0.0255" iyz="0.0" izz="0.0510" />
     </inertial>
-      <collision>
+    <collision>
       <geometry>
         <mesh filename="file:///$(find lunabot_description)/meshes/wheel_link.stl" />
@@ -175,8 +221,20 @@
     </collision>
   </link>
-        <gazebo reference="rear_right_wheel_link">
+  <gazebo reference="rear_right_wheel_link">
     <material>Gazebo/DarkGrey</material>
-  </gazebo>
-    <link name="rear_left_wheel_link">
+    <mu>1.0</mu>
+    <mu2>1.0</mu2>
+    <surface>
+      <contact>
+        <ode>
+          <kp>1000000</kp>
+          <kd>500</kd>
+          <slip1>0.02</slip1>
+          <slip2>0.02</slip2>
+        </ode>
+      </contact>
+    </surface>
+  </gazebo>
+  <link name="rear_left_wheel_link">
     <visual>
       <geometry>
@@ -187,9 +245,9 @@
     </visual>
     <inertial>
-      <mass value="0.1" />
+      <mass value="2.27" />
       <origin xyz="0 0 0" />
-      <inertia ixx="0.01" ixy="0.0" ixz="0.0" iyy="0.01" iyz="0.0" izz="0.01" />
+      <inertia ixx="0.0255" ixy="0.0" ixz="0.0" iyy="0.0255" iyz="0.0" izz="0.0510" />
     </inertial>
-              <collision>
+    <collision>
       <geometry>
         <mesh filename="file:///$(find lunabot_description)/meshes/wheel_link.stl" />
@@ -200,131 +258,112 @@
   <gazebo reference="rear_left_wheel_link">
     <material>Gazebo/DarkGrey</material>
-  </gazebo>
- 	<joint name="base_rear_right_wheel_joint"
-		type="continuous">
-		<parent link="base_link" />
-		<child link="rear_right_wheel_link" />
-		<origin xyz="-0.19 -0.25 0.085"
-			rpy="0 0 0" />
-		<axis xyz="0 1 0" />
-	</joint>
-	<joint name="base_rear_left_wheel_joint"
-		type="continuous">
-		<parent link="base_link" />
-		<child link="rear_left_wheel_link" />
-		<origin xyz="-0.19 0.25 0.085"
-			rpy="0 0 0" />
-		<axis xyz="0 1 0" />
-	</joint>
-	<joint name="base_front_right_wheel_joint"
-		type="continuous">
-		<parent link="base_link" />
-		<child link="front_right_wheel_link" />
-		<origin xyz="0.28 -0.25 0.085"
-			rpy="0 0 0" />
-      <axis xyz="0 1 0" />
-	</joint>
-	<joint name="base_front_left_wheel_joint"
-		type="continuous">
-		<parent link="base_link" />
-		<child link="front_left_wheel_link" />
-		<origin xyz="0.28 0.25 0.085"
-			rpy="0 0 0" />
-      <axis xyz="0 1 0" />
-	</joint>
-	<joint name="base_lidar1_joint"
-		type="fixed">
-		<parent link="base_link" />
-		<child link="lidar1_link" />
-		<origin xyz="0.3630625 0 0.105" rpy="0 0 0" />
-	</joint>
-	<joint name="base_lidar2_joint"
-		type="fixed">
-		<parent link="base_link" />
-		<child link="lidar2_link" />
-		<origin xyz="-0.3630625 0 0.12" rpy="0 0 ${pi}" />
-	</joint>
-	<joint name="base_ebox_link"
-		type="fixed">
-		<parent link="base_link" />
-		<child link="ebox_link" />
-		<origin xyz="0.04 0 0.21" rpy="0 0 0" />
-	</joint>
-	<joint name="base_d455_joint"
-		type="fixed">
-		<parent link="base_link" />
-		<child link="d455_link" />
-		<origin xyz="0.1852625 0.1 0.2"
-			rpy="0 0 0" />
-	</joint>
-	<joint name="base_nuc_joint"
-		type="fixed">
-		<parent link="base_link" />
-		<child link="nuc_link" />
-		<origin xyz="-0.12 0.0 0.145"
-			rpy="0 0 0" />
-	</joint>
-    <joint name="d455_optical_joint" type="fixed">
-        <parent link="d455_link"/>
-        <child link="d455_link_optical"/>
-        <origin xyz="0 0 0" rpy="-1.5708 0 -1.5708"/>
-    </joint>
-   <!-- Differential Drive Plugin -->
-<gazebo>
-  <plugin name="differential_drive_controller" filename="libgazebo_ros_diff_drive.so">
-    <update_rate>50</update_rate>
-    <num_wheel_pairs>2</num_wheel_pairs>
-    <left_joint>base_rear_left_wheel_joint</left_joint>
-    <left_joint>base_front_left_wheel_joint</left_joint>
-    <right_joint>base_rear_right_wheel_joint</right_joint>
-    <right_joint>base_front_right_wheel_joint</right_joint>
-    <wheel_separation>0.5</wheel_separation>
-    <wheel_diameter>0.3</wheel_diameter>
-    <max_wheel_torque>20</max_wheel_torque>
-    <max_wheel_acceleration>1.0</max_wheel_acceleration>
-    <publish_odom>true</publish_odom>
-    <publish_odom_tf>true</publish_odom_tf>
-    <publish_wheel_tf>true</publish_wheel_tf>
-    <odometry_frame>odom</odometry_frame>
-    <robot_base_frame>base_link</robot_base_frame>
-    <command_topic>cmd_vel</command_topic>
-    <ros>
-        <remapping>/odom:=/odometry/filtered</remapping>
-    </ros>
-  </plugin>
-  </gazebo>
+    <mu>1.0</mu>
+    <mu2>1.0</mu2>
+    <surface>
+      <contact>
+        <ode>
+          <kp>1000000</kp>
+          <kd>500</kd>
+          <slip1>0.02</slip1>
+          <slip2>0.02</slip2>
+        </ode>
+      </contact>
+    </surface>
+  </gazebo>
+  <joint name="base_rear_right_wheel_joint" type="continuous">
+    <parent link="base_link" />
+    <child link="rear_right_wheel_link" />
+    <origin xyz="-0.19 -0.25 0.085" rpy="0 0 0" />
+    <axis xyz="0 1 0" />
+  </joint>
+  <joint name="base_rear_left_wheel_joint" type="continuous">
+    <parent link="base_link" />
+    <child link="rear_left_wheel_link" />
+    <origin xyz="-0.19 0.25 0.085" rpy="0 0 0" />
+    <axis xyz="0 1 0" />
+  </joint>
+  <joint name="base_front_right_wheel_joint" type="continuous">
+    <parent link="base_link" />
+    <child link="front_right_wheel_link" />
+    <origin xyz="0.28 -0.25 0.085" rpy="0 0 0" />
+    <axis xyz="0 1 0" />
+  </joint>
+  <joint name="base_front_left_wheel_joint" type="continuous">
+    <parent link="base_link" />
+    <child link="front_left_wheel_link" />
+    <origin xyz="0.28 0.25 0.085" rpy="0 0 0" />
+    <axis xyz="0 1 0" />
+  </joint>
+  <joint name="base_lidar1_joint" type="fixed">
+    <parent link="base_link" />
+    <child link="lidar1_link" />
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
File: lunabot_description/urdf/test_bot.xacro (robot description, xacro)
@@ -8,6 +8,5 @@
 				<mesh filename="file:///$(find lunabot_description)/meshes/base_link.stl" />
 			</geometry>
-			<origin xyz="0 0 0.085"
-				rpy="0 0 0" />
+			<origin xyz="0 0 0.085" rpy="0 0 0" />
 			<material name="light_grey" />
 		</visual>
@@ -18,6 +17,5 @@
 				<mesh filename="file:///$(find lunabot_description)/meshes/ebox_link.stl" />
 			</geometry>
-			<origin xyz="0 0 0"
-				rpy="0 0 0" />
+			<origin xyz="0 0 0" rpy="0 0 0" />
 			<material name="white" />
 		</visual>
@@ -28,6 +26,5 @@
 				<mesh filename="file:///$(find lunabot_description)/meshes/wheel_link.stl" />
 			</geometry>
-			<origin xyz="0 0 0"
-				rpy="${pi / 2.0} 0 0" />
+			<origin xyz="0 0 0" rpy="${pi / 2.0} 0 0" />
 			<material name="green" />
 		</visual>
@@ -38,6 +35,5 @@
 				<mesh filename="file:///$(find lunabot_description)/meshes/wheel_link.stl" />
 			</geometry>
-			<origin xyz="0 0 0"
-				rpy="${-pi / 2.0} 0 0" />
+			<origin xyz="0 0 0" rpy="${-pi / 2.0} 0 0" />
 			<material name="green" />
 		</visual>
@@ -48,6 +44,5 @@
 				<mesh filename="file:///$(find lunabot_description)/meshes/wheel_link.stl" />
 			</geometry>
-			<origin xyz="0 0 0"
-				rpy="${pi / 2.0} 0 0" />
+			<origin xyz="0 0 0" rpy="${pi / 2.0} 0 0" />
 			<material name="green" />
 		</visual>
@@ -58,6 +53,5 @@
 				<mesh filename="file:///$(find lunabot_description)/meshes/wheel_link.stl" />
 			</geometry>
-			<origin xyz="0 0 0"
-				rpy="${-pi / 2.0} 0 0" />
+			<origin xyz="0 0 0" rpy="${-pi / 2.0} 0 0" />
 			<material name="green" />
 		</visual>
@@ -68,6 +62,5 @@
 				<mesh filename="file:///$(find lunabot_description)/meshes/lidar1_link.stl" />
 			</geometry>
-			<origin xyz="0 0 0"
-				rpy="0 0 ${pi / 2.0}" />
+			<origin xyz="0 0 0" rpy="0 0 ${pi / 2.0}" />
 			<material name="black" />
 		</visual>
@@ -78,6 +71,5 @@
 				<mesh filename="file:///$(find lunabot_description)/meshes/lidar2_link.stl" />
 			</geometry>
-			<origin xyz="0 0 0"
-				rpy="0 ${pi} 0" />
+			<origin xyz="0 0 0" rpy="0 ${pi} 0" />
 			<material name="black" />
 		</visual>
@@ -88,6 +80,5 @@
 				<mesh filename="file:///$(find lunabot_description)/meshes/camera_link.stl" />
 			</geometry>
-			<origin xyz="0 0.305 0"
-				rpy="0 0 0" />
+			<origin xyz="0 0.305 0" rpy="0 0 0" />
 			<material name="camera_grey" />
 		</visual>
@@ -98,70 +89,54 @@
 				<mesh filename="file:///$(find lunabot_description)/meshes/nuc_link.stl" />
 			</geometry>
-			<origin xyz="0 0 0"
-				rpy="${pi} 0 ${pi}" />
+			<origin xyz="0 0 0" rpy="${pi} 0 ${pi}" />
 			<material name="black" />
 		</visual>
 	</link>
-	<joint name="base_rear_right_wheel_joint"
-		type="fixed">
+	<joint name="base_rear_right_wheel_joint" type="fixed">
 		<parent link="base_link" />
 		<child link="rear_right_wheel_link" />
-		<origin xyz="-0.19 -0.25 0.085"
-			rpy="0 0 0" />
+		<origin xyz="-0.19 -0.25 0.085" rpy="0 0 0" />
 		<axis xyz="0 1 0" />
 	</joint>
-	<joint name="base_rear_left_wheel_joint"
-		type="fixed">
+	<joint name="base_rear_left_wheel_joint" type="fixed">
 		<parent link="base_link" />
 		<child link="rear_left_wheel_link" />
-		<origin xyz="-0.19 0.25 0.085"
-			rpy="0 0 0" />
+		<origin xyz="-0.19 0.25 0.085" rpy="0 0 0" />
 		<axis xyz="0 1 0" />
 	</joint>
-	<joint name="base_front_right_wheel_joint"
-		type="fixed">
+	<joint name="base_front_right_wheel_joint" type="fixed">
 		<parent link="base_link" />
 		<child link="front_right_wheel_link" />
-		<origin xyz="0.28 -0.25 0.085"
-			rpy="0 0 0" />
+		<origin xyz="0.28 -0.25 0.085" rpy="0 0 0" />
 	</joint>
-	<joint name="base_front_left_wheel_joint"
-		type="fixed">
+	<joint name="base_front_left_wheel_joint" type="fixed">
 		<parent link="base_link" />
 		<child link="front_left_wheel_link" />
-		<origin xyz="0.28 0.25 0.085"
-			rpy="0 0 0" />
+		<origin xyz="0.28 0.25 0.085" rpy="0 0 0" />
 	</joint>
-	<joint name="base_lidar1_joint"
-		type="fixed">
+	<joint name="base_lidar1_joint" type="fixed">
 		<parent link="base_link" />
 		<child link="lidar1_link" />
 		<origin xyz="0 0 0.71" rpy="0 0 ${pi}" />
 	</joint>
-	<joint name="base_lidar2_joint"
-		type="fixed">
+	<joint name="base_lidar2_joint" type="fixed">
 		<parent link="base_link" />
 		<child link="lidar2_link" />
 		<origin xyz="0.305 0 0.12" rpy="0 ${pi} 0" />
 	</joint>
-	<joint name="base_ebox_link"
-		type="fixed">
+	<joint name="base_ebox_link" type="fixed">
 		<parent link="base_link" />
 		<child link="ebox_link" />
 		<origin xyz="0.04 0 0.21" rpy="0 0 0" />
 	</joint>
-	<joint name="base_d455_joint"
-		type="fixed">
+	<joint name="base_d455_joint" type="fixed">
 		<parent link="base_link" />
 		<child link="d455_link" />
-		<origin xyz="0.305 0.1 0.2"
-			rpy="0 0 0" />
+		<origin xyz="0.305 0.1 0.2" rpy="0 0 0" />
 	</joint>
-	<joint name="base_nuc_joint"
-		type="fixed">
+	<joint name="base_nuc_joint" type="fixed">
 		<parent link="base_link" />
 		<child link="nuc_link" />
-		<origin xyz="-0.12 0.0 0.145"
-			rpy="0 0 0" />
+		<origin xyz="-0.12 0.0 0.145" rpy="0 0 0" />
 	</joint>
 </robot>
