Commit message: Changed folder structure, trying to get mapping working with simulation but ekf_node is acting strange.

File: lunabot_simulation/urdf/sim_bot.xacro (robot description, xacro)
@@ -6,5 +6,5 @@
     <visual>
       <geometry>
-        <mesh filename="file:///$(find lunabot_description)/meshes/base_link.stl" />
+        <mesh filename="file:///$(find lunabot_simulation)/meshes/base_link.stl" />
       </geometry>
       <origin xyz="0 0 0.085" rpy="0 0 0" />
@@ -13,5 +13,5 @@
     <collision>
       <geometry>
-        <mesh filename="file:///$(find lunabot_description)/meshes/base_link.stl" />
+        <mesh filename="file:///$(find lunabot_simulation)/meshes/base_link.stl" />
       </geometry>
       <origin xyz="0 0 0.085" rpy="0 0 0" />
@@ -29,5 +29,5 @@
     <visual>
       <geometry>
-        <mesh filename="file:///$(find lunabot_description)/meshes/ebox_link.stl" />
+        <mesh filename="file:///$(find lunabot_simulation)/meshes/ebox_link.stl" />
       </geometry>
       <origin xyz="0 0 0" rpy="0 0 0" />
@@ -36,5 +36,5 @@
     <collision>
       <geometry>
-        <mesh filename="file:///$(find lunabot_description)/meshes/ebox_link.stl" />
+        <mesh filename="file:///$(find lunabot_simulation)/meshes/ebox_link.stl" />
       </geometry>
       <origin xyz="0 0 0" rpy="0 0 0" />
@@ -47,5 +47,5 @@
     <visual>
       <geometry>
-        <mesh filename="file:///$(find lunabot_description)/meshes/nuc_link.stl" />
+        <mesh filename="file:///$(find lunabot_simulation)/meshes/nuc_link.stl" />
       </geometry>
       <origin xyz="0 0 0" rpy="${pi} 0 ${pi}" />
@@ -54,5 +54,5 @@
     <collision>
       <geometry>
-        <mesh filename="file:///$(find lunabot_description)/meshes/nuc_link.stl" />
+        <mesh filename="file:///$(find lunabot_simulation)/meshes/nuc_link.stl" />
       </geometry>
       <origin xyz="0 0 0" rpy="${pi} 0 ${pi}" />
@@ -65,5 +65,5 @@
     <visual>
       <geometry>
-        <mesh filename="file:///$(find lunabot_description)/meshes/lidar1_link.stl" />
+        <mesh filename="file:///$(find lunabot_simulation)/meshes/lidar1_link.stl" />
       </geometry>
       <origin xyz="0 0 0" rpy="0 0 -1.5708" />
@@ -72,5 +72,5 @@
     <collision>
       <geometry>
-        <mesh filename="file:///$(find lunabot_description)/meshes/lidar1_link.stl" />
+        <mesh filename="file:///$(find lunabot_simulation)/meshes/lidar1_link.stl" />
       </geometry>
       <origin xyz="0 0 0" rpy="0 0 -1.5708" />
@@ -80,5 +80,5 @@
     <visual>
       <geometry>
-        <mesh filename="file:///$(find lunabot_description)/meshes/blade_link.stl" />
+        <mesh filename="file:///$(find lunabot_simulation)/meshes/blade_link.stl" />
       </geometry>
       <origin xyz="0 0 0" rpy="0 0 0" />
@@ -87,5 +87,5 @@
     <collision>
       <geometry>
-        <mesh filename="file:///$(find lunabot_description)/meshes/blade_link.stl" />
+        <mesh filename="file:///$(find lunabot_simulation)/meshes/blade_link.stl" />
       </geometry>
       <origin xyz="0 0 0" rpy="0 0 0" />
@@ -103,5 +103,5 @@
     <visual>
       <geometry>
-        <mesh filename="file:///$(find lunabot_description)/meshes/lidar2_link.stl" />
+        <mesh filename="file:///$(find lunabot_simulation)/meshes/lidar2_link.stl" />
       </geometry>
       <origin xyz="0 0 0" rpy="0 0 0" />
@@ -110,13 +110,13 @@
     <collision>
       <geometry>
-        <mesh filename="file:///$(find lunabot_description)/meshes/lidar2_link.stl" />
-      </geometry>
-      <origin xyz="0 0 0" rpy="0 0 0" />
-    </collision>
-  </link>
-  <link name="d455_link">
-    <visual>
-      <geometry>
-        <mesh filename="file:///$(find lunabot_description)/meshes/camera_link.stl" />
+        <mesh filename="file:///$(find lunabot_simulation)/meshes/lidar2_link.stl" />
+      </geometry>
+      <origin xyz="0 0 0" rpy="0 0 0" />
+    </collision>
+  </link>
+  <link name="d456_link">
+    <visual>
+      <geometry>
+        <mesh filename="file:///$(find lunabot_simulation)/meshes/camera_link.stl" />
       </geometry>
       <origin xyz="0 0 0" rpy="0 0 0" />
@@ -125,14 +125,15 @@
     <collision>
       <geometry>
-        <mesh filename="file:///$(find lunabot_description)/meshes/camera_link.stl" />
-      </geometry>
-      <origin xyz="0 0 0" rpy="0 0 0" />
-    </collision>
-  </link>
-  <link name="d455_link_optical"></link>
+        <mesh filename="file:///$(find lunabot_simulation)/meshes/camera_link.stl" />
+      </geometry>
+      <origin xyz="0 0 0" rpy="0 0 0" />
+    </collision>
+  </link>
+  <link name="d456_link_optical"></link>
+  <link name="imu_link"></link>
   <link name="front_right_wheel_link">
     <visual>
       <geometry>
-        <mesh filename="file:///$(find lunabot_description)/meshes/wheel_link.stl" />
+        <mesh filename="file:///$(find lunabot_simulation)/meshes/wheel_link.stl" />
       </geometry>
       <origin xyz="0 0 0" rpy="1.5708 0 0" />
@@ -143,8 +144,8 @@
       <origin xyz="0 0 0" />
       <inertia ixx="0.0255" ixy="0.0" ixz="0.0" iyy="0.0255" iyz="0.0" izz="0.0510" />
-></inertial>
-    <collision>
-      <geometry>
-        <mesh filename="file:///$(find lunabot_description)/meshes/wheel_link.stl" />
+    </inertial>
+    <collision>
+      <geometry>
+        <mesh filename="file:///$(find lunabot_simulation)/meshes/wheel_link.stl" />
       </geometry>
       <origin xyz="0 0 0" rpy="1.5708 0 0" />
@@ -169,5 +170,5 @@
     <visual>
       <geometry>
-        <mesh filename="file:///$(find lunabot_description)/meshes/wheel_link.stl" />
+        <mesh filename="file:///$(find lunabot_simulation)/meshes/wheel_link.stl" />
       </geometry>
       <origin xyz="0 0 0" rpy="-1.5708 0 0" />
@@ -181,5 +182,5 @@
     <collision>
       <geometry>
-        <mesh filename="file:///$(find lunabot_description)/meshes/wheel_link.stl" />
+        <mesh filename="file:///$(find lunabot_simulation)/meshes/wheel_link.stl" />
       </geometry>
       <origin xyz="0 0 0" rpy="-1.5708 0 0" />
@@ -204,5 +205,5 @@
     <visual>
       <geometry>
-        <mesh filename="file:///$(find lunabot_description)/meshes/wheel_link.stl" />
+        <mesh filename="file:///$(find lunabot_simulation)/meshes/wheel_link.stl" />
       </geometry>
       <origin xyz="0 0 0" rpy="1.5708 0 0" />
@@ -216,5 +217,5 @@
     <collision>
       <geometry>
-        <mesh filename="file:///$(find lunabot_description)/meshes/wheel_link.stl" />
+        <mesh filename="file:///$(find lunabot_simulation)/meshes/wheel_link.stl" />
       </geometry>
       <origin xyz="0 0 0" rpy="1.5708 0 0" />
@@ -239,5 +240,5 @@
     <visual>
       <geometry>
-        <mesh filename="file:///$(find lunabot_description)/meshes/wheel_link.stl" />
+        <mesh filename="file:///$(find lunabot_simulation)/meshes/wheel_link.stl" />
       </geometry>
       <origin xyz="0 0 0" rpy="-1.5708 0 0" />
@@ -251,5 +252,5 @@
     <collision>
       <geometry>
-        <mesh filename="file:///$(find lunabot_description)/meshes/wheel_link.stl" />
+        <mesh filename="file:///$(find lunabot_simulation)/meshes/wheel_link.stl" />
       </geometry>
       <origin xyz="0 0 0" rpy="-1.5708 0 0" />
@@ -323,16 +324,21 @@
     <dynamics damping="0.0" friction="0.0" />
   </joint>
-  <joint name="base_d455_joint" type="fixed">
-    <parent link="base_link" />
-    <child link="d455_link" />
+  <joint name="base_d456_joint" type="fixed">
+    <parent link="base_link" />
+    <child link="d456_link" />
     <origin xyz="0.1602565 0 0.355" rpy="0 0 0" />
   </joint>
-  <joint name="d455_optical_joint" type="fixed">
-    <parent link="d455_link" />
-    <child link="d455_link_optical" />
+  <joint name="d456_optical_joint" type="fixed">
+    <parent link="d456_link" />
+    <child link="d456_link_optical" />
     <origin xyz="0 0 0" rpy="-1.5708 0 -1.5708" />
   </joint>
-  <gazebo reference="d455_link">
-    <sensor type="depth" name="d455">
+  <joint name="imu_joint" type="fixed">
+    <parent link="base_link"/>
+    <child link="imu_link"/>
+    <origin xyz="0 0 0" rpy="0 0 0"/>
+  </joint>
+  <gazebo reference="d456_link">
+    <sensor type="depth" name="d456">
       <pose>0 0 0 0 0 0</pose>
       <visualize>true</visualize>
@@ -352,11 +358,11 @@
       <plugin name="camera_controller" filename="libgazebo_ros_camera.so">
         <ros>
-          <remapping>/d455/image_raw:=/d455/color/image_raw</remapping>
-          <remapping>/d455/points:=/d455/color/points</remapping>
-          <remapping>/d455/camera_info:=/d455/color/camera_info</remapping>
-          <remapping>/d455/depth/image_raw:=/d455/depth/image_rect_raw</remapping>
+          <remapping>/d456/image_raw:=/d456/color/image_raw</remapping>
+          <remapping>/d456/points:=/d456/color/points</remapping>
+          <remapping>/d456/camera_info:=/d456/color/camera_info</remapping>
+          <remapping>/d456/depth/image_raw:=/d456/depth/image_rect_raw</remapping>
           <update_rate>30.0</update_rate>
         </ros>
-        <frame_name>d455_link_optical</frame_name>
+        <frame_name>d456_link_optical</frame_name>
       </plugin>
     </sensor>
@@ -364,13 +370,13 @@
   </gazebo>
   <gazebo reference="lidar1_link">
-    <sensor type="ray" name="lidar1">
+    <sensor type="ray" name="lidar1_link">
       <pose>0 0 0 0 0 0</pose>
       <visualize>false</visualize>
-      <update_rate>30.0</update_rate>
+      <update_rate>50.0</update_rate>
       <ray>
         <scan>
           <horizontal>
-            <samples>720</samples>
-            <resolution>1</resolution>
+            <samples>1080</samples>
+            <resolution>0.5</resolution>
             <min_angle>-3.14</min_angle>
             <max_angle>3.14</max_angle>
@@ -378,9 +384,14 @@
         </scan>
         <range>
-          <min>0.05</min>
-          <max>12.0</max>
+          <min>0.1</min>
+          <max>10.0</max>
         </range>
+        <noise>
+          <type>gaussian</type>
+          <mean>0.0</mean>
+          <stddev>0.01</stddev>
+        </noise>
       </ray>
-      <plugin name="lidar1_controller" filename="libgazebo_ros_ray_sensor.so">
+      <plugin name="lidar1_controller" filename="libgazebo_ros_ray_sensor.so">        <!-- GPU plugin for performance -->
         <frame_name>lidar1_link</frame_name>
         <ros>
@@ -393,31 +404,58 @@
   </gazebo>
   <gazebo reference="lidar2_link">
-    <sensor type="ray" name="lidar2">
+    <sensor type="ray" name="lidar2_link">
       <pose>0 0 0 0 0 0</pose>
       <visualize>false</visualize>
-      <update_rate>30.0</update_rate>
+      <update_rate>50.0</update_rate>
       <ray>
         <scan>
           <horizontal>
-            <samples>720</samples>
-            <resolution>1</resolution>
-            <min_angle>-1.5708</min_angle>
-            <max_angle>1.5708</max_angle>
+            <samples>1080</samples>
+            <resolution>0.5</resolution>
+            <min_angle>-1.57</min_angle>
+            <max_angle>1.57</max_angle>
           </horizontal>
         </scan>
         <range>
-          <min>0.05</min>
-          <max>12.0</max>
+          <min>0.1</min>
+          <max>10.0</max>
         </range>
+        <noise>
+          <type>gaussian</type>
+          <mean>0.0</mean>
+          <stddev>0.01</stddev>
+        </noise>
       </ray>
       <plugin name="lidar2_controller" filename="libgazebo_ros_ray_sensor.so">
+        <frame_name>lidar2_link</frame_name>
         <ros>
           <remapping>~/out:=/scan2</remapping>
         </ros>
         <output_type>sensor_msgs/LaserScan</output_type>
-        <frame_name>lidar2_link</frame_name>
       </plugin>
     </sensor>
     <material>Gazebo/Black</material>
+  </gazebo>
+  <gazebo reference="imu_link">
+    <gravity>true</gravity>
+    <sensor name="imu_sensor" type="imu">
+      <always_on>true</always_on>
+      <update_rate>100</update_rate>
+      <visualize>true</visualize>
+      <plugin filename="libgazebo_ros_imu_sensor.so" name="imu_plugin">
+        <ros>
+          <namespace></namespace>
+          <remapping>~/out:=/imu/data_raw</remapping>
+        </ros>
+        <bodyName>base_link</bodyName>
+        <updateRateHZ>100.0</updateRateHZ>
+        <gaussianNoise>0.0</gaussianNoise>
+        <xyzOffset>0 0 0</xyzOffset>
+        <rpyOffset>0 0 0</rpyOffset>
+        <frameName>imu_link</frameName>
+        <initialOrientationAsReference>false</initialOrientationAsReference>
+      </plugin>
+      <pose>0 0 0 0 0 0</pose>
+    </sensor>
   </gazebo>
   <ros2_control name="GazeboSystem" type="system">
@@ -467,5 +505,5 @@
       <robot_param>robot_description</robot_param>
       <robot_param_node>robot_state_publisher</robot_param_node>
-      <parameters>$(find lunabot_bringup)/params/sim_params.yaml</parameters>
+      <parameters>$(find lunabot_config)/params/sim_params.yaml</parameters>
     </plugin>
   </gazebo>

File: lunabot_simulation/urdf/test_bot.xacro (robot description, xacro)
@@ -6,5 +6,5 @@
 		<visual>
 			<geometry>
-				<mesh filename="file:///$(find lunabot_description)/meshes/base_link.stl" />
+				<mesh filename="file:///$(find lunabot_simulation)/meshes/base_link.stl" />
 			</geometry>
 			<origin xyz="0 0 0.085" rpy="0 0 0" />
@@ -15,5 +15,5 @@
 		<visual>
 			<geometry>
-				<mesh filename="file:///$(find lunabot_description)/meshes/ebox_link.stl" />
+				<mesh filename="file:///$(find lunabot_simulation)/meshes/ebox_link.stl" />
 			</geometry>
 			<origin xyz="0 0 0" rpy="0 0 0" />
@@ -24,5 +24,5 @@
 		<visual>
 			<geometry>
-				<mesh filename="file:///$(find lunabot_description)/meshes/wheel_link.stl" />
+				<mesh filename="file:///$(find lunabot_simulation)/meshes/wheel_link.stl" />
 			</geometry>
 			<origin xyz="0 0 0" rpy="${pi / 2.0} 0 0" />
@@ -33,5 +33,5 @@
 		<visual>
 			<geometry>
-				<mesh filename="file:///$(find lunabot_description)/meshes/wheel_link.stl" />
+				<mesh filename="file:///$(find lunabot_simulation)/meshes/wheel_link.stl" />
 			</geometry>
 			<origin xyz="0 0 0" rpy="${-pi / 2.0} 0 0" />
@@ -42,5 +42,5 @@
 		<visual>
 			<geometry>
-				<mesh filename="file:///$(find lunabot_description)/meshes/wheel_link.stl" />
+				<mesh filename="file:///$(find lunabot_simulation)/meshes/wheel_link.stl" />
 			</geometry>
 			<origin xyz="0 0 0" rpy="${pi / 2.0} 0 0" />
@@ -51,5 +51,5 @@
 		<visual>
 			<geometry>
-				<mesh filename="file:///$(find lunabot_description)/meshes/wheel_link.stl" />
+				<mesh filename="file:///$(find lunabot_simulation)/meshes/wheel_link.stl" />
 			</geometry>
 			<origin xyz="0 0 0" rpy="${-pi / 2.0} 0 0" />
@@ -60,5 +60,5 @@
 		<visual>
 			<geometry>
-				<mesh filename="file:///$(find lunabot_description)/meshes/lidar1_link.stl" />
+				<mesh filename="file:///$(find lunabot_simulation)/meshes/lidar1_link.stl" />
 			</geometry>
 			<origin xyz="0 0 0" rpy="0 0 ${pi / 2.0}" />
@@ -69,5 +69,5 @@
 		<visual>
 			<geometry>
-				<mesh filename="file:///$(find lunabot_description)/meshes/lidar2_link.stl" />
+				<mesh filename="file:///$(find lunabot_simulation)/meshes/lidar2_link.stl" />
 			</geometry>
 			<origin xyz="0 0 0" rpy="0 ${pi} 0" />
@@ -75,8 +75,8 @@
 		</visual>
 	</link>
-	<link name="d455_link">
+	<link name="d456_link">
 		<visual>
 			<geometry>
-				<mesh filename="file:///$(find lunabot_description)/meshes/camera_link.stl" />
+				<mesh filename="file:///$(find lunabot_simulation)/meshes/camera_link.stl" />
 			</geometry>
 			<origin xyz="0 0.305 0" rpy="0 0 0" />
@@ -87,5 +87,5 @@
 		<visual>
 			<geometry>
-				<mesh filename="file:///$(find lunabot_description)/meshes/nuc_link.stl" />
+				<mesh filename="file:///$(find lunabot_simulation)/meshes/nuc_link.stl" />
 			</geometry>
 			<origin xyz="0 0 0" rpy="${pi} 0 ${pi}" />
@@ -130,7 +130,7 @@
 		<origin xyz="0.04 0 0.21" rpy="0 0 0" />
 	</joint>
-	<joint name="base_d455_joint" type="fixed">
+	<joint name="base_d456_joint" type="fixed">
 		<parent link="base_link" />
-		<child link="d455_link" />
+		<child link="d456_link" />
 		<origin xyz="0.305 0.1 0.2" rpy="0 0 0" />
 	</joint>

Commit message: Updated dependencies and parameters, changed speed of robot in simulation.

File: lunabot_simulation/urdf/sim_bot.xacro (robot description, xacro)
@@ -327,5 +327,5 @@
     <parent link="base_link" />
     <child link="d456_link" />
-    <origin xyz="0.1602565 0 0.355" rpy="0 0 0" />
+    <origin xyz="0.1602565 0 0.8" rpy="0 0 0" />
   </joint>
   <joint name="d456_optical_joint" type="fixed">
@@ -353,5 +353,5 @@
         <clip>
           <near>0.05</near>
-          <far>5.0</far>
+          <far>10.0</far>
         </clip>
       </camera>
@@ -441,5 +441,5 @@
     <sensor name="imu_sensor" type="imu">
       <always_on>true</always_on>
-      <update_rate>100</update_rate>
+      <update_rate>50</update_rate>
       <visualize>true</visualize>
       <plugin filename="libgazebo_ros_imu_sensor.so" name="imu_plugin">

Commit message: Updated README.md, dependencies, and camera height in sim_bot.xacro

File: lunabot_simulation/urdf/sim_bot.xacro (robot description, xacro)
@@ -327,5 +327,5 @@
     <parent link="base_link" />
     <child link="d456_link" />
-    <origin xyz="0.1602565 0 0.8" rpy="0 0 0" />
+    <origin xyz="0.1602565 0 0.6" rpy="0 0 0" />
   </joint>
   <joint name="d456_optical_joint" type="fixed">
