Commit message: Added Falcon 500 support for testing on last years' robot

File: lunabot_simulation/urdf/bulldozer_bot.xacro (robot description, xacro)
@@ -239,5 +239,5 @@
     <parent link="base_link" />
     <child link="lidar1_link" />
-    <origin xyz="-0.0925 0 0.4575" rpy="0 0 0" />
+    <origin xyz="-0.0925 0 0.6075" rpy="0 0 0" />
   </joint>
   <joint name="base_lidar2_joint" type="fixed">
@@ -262,5 +262,5 @@
     <parent link="base_link" />
     <child link="d455_link" />
-    <origin xyz="-0.12 0 0.40" rpy="0 0 0" />
+    <origin xyz="-0.12 0 0.55" rpy="0 0 0" />
   </joint>
   <joint name="d455_optical_joint" type="fixed">
@@ -272,10 +272,10 @@
     <parent link="base_link" />
     <child link="d456_link" />
-    <origin xyz="0.29 0 0.35" rpy="0 0.261799 0" />
+    <origin xyz="-0.05 0 0.55" rpy="0 0.523599 0" />
   </joint>
   <joint name="d456_optical_joint" type="fixed">
     <parent link="d456_link" />
     <child link="d456_optical_link" />
-    <origin xyz="0 0 0" rpy="-1.309001 0 -1.5708" />
+    <origin xyz="0 0 0" rpy="-1.047201 0 -1.5708" />
   </joint>
   <joint name="imu_joint" type="fixed">
@@ -393,5 +393,5 @@
   <gazebo reference="d456_link">
     <sensor type="depth" name="d456">
-      <pose>0 0 0 0 -0.261799 0</pose>
+      <pose>0 0 0 0 -0.523599 0</pose>
       <update_rate>60.0</update_rate>
       <visualize>true</visualize>
