Commit message: Fixed parameter issues with real_launch

File: lunabot_simulation/urdf/real_bot.xacro (robot description, xacro)
@@ -104,5 +104,5 @@
         <mesh filename="file:///$(find lunabot_simulation)/meshes/camera_link.stl" />
       </geometry>
-      <origin xyz="0 0 0" rpy="0 0 0" />
+      <origin xyz="0 0 0" rpy="0 0 3.14" />
       <material name="camera_grey" />
     </visual>
@@ -111,5 +111,5 @@
         <mesh filename="file:///$(find lunabot_simulation)/meshes/camera_link.stl" />
       </geometry>
-      <origin xyz="0 0 0" rpy="0 0 0" />
+      <origin xyz="0 0 0" rpy="0 0 3.14" />
     </collision>
   </link>
@@ -259,10 +259,10 @@
     <parent link="base_link" />
     <child link="d455_link" />
-    <origin xyz="-0.12 0 0.55" rpy="0 0 0" />
+    <origin xyz="-0.305 0 0.45" rpy="0 0 3.14" />
   </joint>
   <joint name="base_d456_joint" type="fixed">
     <parent link="base_link" />
     <child link="d456_link" />
-    <origin xyz="-0.05 0 0.55" rpy="0 0.523599 0" />
+    <origin xyz="0.305 0 0.55" rpy="0 0 0" />
   </joint>
 </robot>
